Commit message: rotation perfectly stable
updated wrench_movement's pose callback and robosub's urdf file

File: high_level_robosub/urdf/high_level_robosub.urdf (robot description, URDF)
Before this commit: robot high_level_robosub, 2 links, 1 joints
Links:
- added link bouyant_link, mass 50.0; collision box size=0.7 0.7 0.4; visual box size=0.7 0.7 0.1
- link base_link: mass 200.0 -> 350.0; geometry collision box size=0.7 0.7 0.4; visual box size=0.7 0.7 0.4
- link camera_link: mass 1.0 -> None
Joints:
- added joint bouyant_joint: type fixed, parent base_link, child bouyant_link, origin xyz=0 0 0.25 rpy=0 0 0
- joint camera_joint: origin xyz=0.358 0 0 rpy=3.1416 3.1416 3.1416 -> xyz=0.35 0 0 rpy=3.1416 3.1416 3.1416
